File: PCB Design/Rev 2/Tilt_Table_PCB_Rev2/power_conversion.kicad_sch (KiCad schematic)
At the start: 14 parts, among them J5 BUCK_EN, U4 TPS54531DDA

Commit message: PCB Rev 2 Update
Parts:
- renumbered C17 to C10, C19 to C11, C20 to C12, C27 to C13, C29 to C14, C31 to C15, C16 to C9, D5 to D3, J5 to J4, L2 to L1, R22 to R19, R25 to R20, R26 to R21, U4 to U2
Other:
- company: (none) -> Made by Jasper Tan
- title: (none) -> Tilt Plate Board
Changed lines of the file:
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@@
 	(generator_version "9.0")
 	(paper "A4")
+	(title_block
+		(title "Tilt Plate Board")
+		(date "2026-04-25")
+		(rev "2.0")
+		(company "Made by Jasper Tan")
+	)
 	(rectangle
 		(start 38.1 33.02)
@@
 		(dnp no)
 		(fields_autoplaced yes)
-		(property "Reference" "#PWR065"
+		(property "Reference" "#PWR032"
 			(at 157.48 77.47 0)
 			(effects
@@
 			(project "Tilt_Table_PCB_Rev2"
 				(path "/1c736c1b-ed9d-403f-bc84-83343cfbb355/4372dc6b-a760-44d8-8e04-eabd010a5ae9"
-					(reference "#PWR065")
+					(reference "#PWR032")
 					(unit 1)
 				)
@@
 		(on_board yes)
 		(dnp no)
-		(property "Reference" "C16"
+		(property "Reference" "C9"
 			(at 40.64 50.8 0)
 			(effects
@@
 			(project "Tilt_Table_PCB_Rev2"
 				(path "/1c736c1b-ed9d-403f-bc84-83343cfbb355/4372dc6b-a760-44d8-8e04-eabd010a5ae9"
-					(reference "C16")
+					(reference "C9")
 					(unit 1)
 				)
@@
 		(dnp no)
 		(fields_autoplaced yes)
-		(property "Reference" "#PWR048"
+		(property "Reference" "#PWR029"
 			(at 104.14 90.17 0)
 			(effects
@@
 			(project "Tilt_Table_PCB_Rev2"
 				(path "/1c736c1b-ed9d-403f-bc84-83343cfbb355/4372dc6b-a760-44d8-8e04-eabd010a5ae9"
-					(reference "#PWR048")
+					(reference "#PWR029")
 					(unit 1)
 				)
@@
 		(dnp no)
 		(fields_autoplaced yes)
-		(property "Reference" "R26"
+		(property "Reference" "R21"
 			(at 160.02 66.0399 0)
 			(effects
@@
 			(project "Tilt_Table_PCB_Rev2"
 				(path "/1c736c1b-ed9d-403f-bc84-83343cfbb355/4372dc6b-a760-44d8-8e04-eabd010a5ae9"
-					(reference "R26")
+					(reference "R21")
 					(unit 1)
 				)
@@
 		(on_board yes)
 		(dnp no)
-		(property "Reference" "J5"
+		(property "Reference" "J4"
 			(at 57.15 36.83 0)
 			(effects
@@
 			(project "Tilt_Table_PCB_Rev2"
 				(path "/1c736c1b-ed9d-403f-bc84-83343cfbb355/4372dc6b-a760-44d8-8e04-eabd010a5ae9"
-					(reference "J5")
+					(reference "J4")
 					(unit 1)
 				)
@@
 		(on_board yes)
 		(dnp no)
-		(property "Reference" "C17"
+		(property "Reference" "C10"
 			(at 49.53 85.09 0)
 			(effects
@@
 			(project "Tilt_Table_PCB_Rev2"
 				(path "/1c736c1b-ed9d-403f-bc84-83343cfbb355/4372dc6b-a760-44d8-8e04-eabd010a5ae9"
-					(reference "C17")
+					(reference "C10")
 					(unit 1)
 				)
@@
 		(dnp no)
 		(fields_autoplaced yes)
-		(property "Reference" "#PWR040"
+		(property "Reference" "#PWR027"
 			(at 66.04 69.85 0)
 			(effects
@@
 			(project "Tilt_Table_PCB_Rev2"
 				(path "/1c736c1b-ed9d-403f-bc84-83343cfbb355/4372dc6b-a760-44d8-8e04-eabd010a5ae9"
-					(reference "#PWR040")
+					(reference "#PWR027")
 					(unit 1)
 				)
@@
 		(dnp no)
 		(fields_autoplaced yes)
-		(property "Reference" "#PWR042"
+		(property "Reference" "#PWR028"
 			(at 67.31 100.33 0)
 			(effects
@@
 			(project "Tilt_Table_PCB_Rev2"
 				(path "/1c736c1b-ed9d-403f-bc84-83343cfbb355/4372dc6b-a760-44d8-8e04-eabd010a5ae9"
-					(reference "#PWR042")
+					(reference "#PWR028")
 					(unit 1)
 				)
@@
 		(dnp no)
 		(fields_autoplaced yes)
-		(property "Reference" "#PWR036"
+		(property "Reference" "#PWR026"
 			(at 46.99 62.23 0)
 			(effects
@@
 			(project "Tilt_Table_PCB_Rev2"
 				(path "/1c736c1b-ed9d-403f-bc84-83343cfbb355/4372dc6b-a760-44d8-8e04-eabd010a5ae9"
-					(reference "#PWR036")
+					(reference "#PWR026")
 					(unit 1)
 				)
@@
 		(on_board yes)
 		(dnp no)
-		(property "Reference" "C31"
+		(property "Reference" "C15"
 			(at 148.59 52.07 0)
 			(effects
@@
 			(project "Tilt_Table_PCB_Rev2"
 				(path "/1c736c1b-ed9d-403f-bc84-83343cfbb355/4372dc6b-a760-44d8-8e04-eabd010a5ae9"
-					(reference "C31")
+					(reference "C15")
 					(unit 1)
 				)
@@
 		(on_board yes)
 		(dnp no)
-		(property "Reference" "#FLG04"
+		(property "Reference" "#FLG02"
 			(at 137.16 46.355 0)
 			(effects
@@
 			(project "Tilt_Table_PCB_Rev2"
 				(path "/1c736c1b-ed9d-403f-bc84-83343cfbb355/4372dc6b-a760-44d8-8e04-eabd010a5ae9"
-					(reference "#FLG04")
+					(reference "#FLG02")
 					(unit 1)
 				)
@@
 		(dnp no)
 		(fields_autoplaced yes)
-		(property "Reference" "R25"
+		(property "Reference" "R20"
 			(at 160.02 57.1499 0)
 			(effects
@@
 			(project "Tilt_Table_PCB_Rev2"
 				(path "/1c736c1b-ed9d-403f-bc84-83343cfbb355/4372dc6b-a760-44d8-8e04-eabd010a5ae9"
-					(reference "R25")
+					(reference "R20")
 					(unit 1)
 				)
@@
 		(on_board yes)
 		(dnp no)
-		(property "Reference" "C20"
+		(property "Reference" "C12"
 			(at 60.96 81.28 0)
 			(effects
@@
 			(project "Tilt_Table_PCB_Rev2"
 				(path "/1c736c1b-ed9d-403f-bc84-83343cfbb355/4372dc6b-a760-44d8-8e04-eabd010a5ae9"
-					(reference "C20")
+					(reference "C12")
 					(unit 1)
 				)
@@
 		(on_board yes)
 		(dnp no)
-		(property "Reference" "C29"
+		(property "Reference" "C14"
 			(at 138.43 52.07 0)
 			(effects
@@
 			(project "Tilt_Table_PCB_Rev2"
 				(path "/1c736c1b-ed9d-403f-bc84-83343cfbb355/4372dc6b-a760-44d8-8e04-eabd010a5ae9"
-					(reference "C29")
+					(reference "C14")
 					(unit 1)
 				)
@@
 		(dnp no)
 		(fields_autoplaced yes)
-		(property "Reference" "#PWR062"
+		(property "Reference" "#PWR031"
 			(at 149.86 52.07 0)
 			(effects
@@
 			(project "Tilt_Table_PCB_Rev2"
 				(path "/1c736c1b-ed9d-403f-bc84-83343cfbb355/4372dc6b-a760-44d8-8e04-eabd010a5ae9"
-					(reference "#PWR062")
+					(reference "#PWR031")
 					(unit 1)
 				)
@@
 		(dnp no)
 		(fields_autoplaced yes)
-		(property "Reference" "L2"
+		(property "Reference" "L1"
 			(at 128.27 43.18 90)
 			(effects
@@
 			(project "Tilt_Table_PCB_Rev2"
 				(path "/1c736c1b-ed9d-403f-bc84-83343cfbb355/4372dc6b-a760-44d8-8e04-eabd010a5ae9"
-					(reference "L2")
+					(reference "L1")
 					(unit 1)
 				)
@@
 		(dnp no)
 		(fields_autoplaced yes)
-		(property "Reference" "#PWR061"
+		(property "Reference" "#PWR030"
 			(at 134.62 63.5 0)
 			(effects
@@
 			(project "Tilt_Table_PCB_Rev2"
 				(path "/1c736c1b-ed9d-403f-bc84-83343cfbb355/4372dc6b-a760-44d8-8e04-eabd010a5ae9"
-					(reference "#PWR061")
+					(reference "#PWR030")
 					(unit 1)
 				)
@@
 		(dnp no)
 		(fields_autoplaced yes)
-		(property "Reference" "D5"
+		(property "Reference" "D3"
 			(at 125.73 52.0699 90)
 			(effects
@@
 			(project "Tilt_Table_PCB_Rev2"
 				(path "/1c736c1b-ed9d-403f-bc84-83343cfbb355/4372dc6b-a760-44d8-8e04-eabd010a5ae9"
-					(reference "D5")
+					(reference "D3")
 					(unit 1)
 				)
@@
 		(dnp no)
 		(fields_autoplaced yes)
-		(property "Reference" "R22"
+		(property "Reference" "R19"
 			(at 69.85 87.6299 0)
 			(effects
@@
 			(project "Tilt_Table_PCB_Rev2"
 				(path "/1c736c1b-ed9d-403f-bc84-83343cfbb355/4372dc6b-a760-44d8-8e04-eabd010a5ae9"
-					(reference "R22")
+					(reference "R19")
 					(unit 1)
 				)
@@
 		(dnp no)
 		(fields_autoplaced yes)
-		(property "Reference" "U4"
+		(property "Reference" "U2"
 			(at 86.36 38.1 0)
 			(effects
@@
 			(project "Tilt_Table_PCB_Rev2"
 				(path "/1c736c1b-ed9d-403f-bc84-83343cfbb355/4372dc6b-a760-44d8-8e04-eabd010a5ae9"
-					(reference "U4")
+					(reference "U2")
 					(unit 1)
 				)
@@
 		(on_board yes)
 		(dnp no)
-		(property "Reference" "C27"
+		(property "Reference" "C13"
 			(at 109.22 40.64 90)
 			(effects
@@
 			(project "Tilt_Table_PCB_Rev2"
 				(path "/1c736c1b-ed9d-403f-bc84-83343cfbb355/4372dc6b-a760-44d8-8e04-eabd010a5ae9"
-					(reference "C27")
+					(reference "C13")
 					(unit 1)
 				)
@@
 		(on_board yes)
 		(dnp no)
-		(property "Reference" "C19"
+		(property "Reference" "C11"
 			(at 59.69 59.69 0)
 			(effects
@@
 			(project "Tilt_Table_PCB_Rev2"
 				(path "/1c736c1b-ed9d-403f-bc84-83343cfbb355/4372dc6b-a760-44d8-8e04-eabd010a5ae9"
-					(reference "C19")
+					(reference "C11")
 					(unit 1)
 				)
